Commit message: pick and place implementation

File: so-arm/so101_ws/src/so101_description/urdf/so101_new_calib.urdf (robot description, URDF)
Before this commit: robot so101_new_calib, 8 links, 7 joints
Links:
- added link camera_color_optical_frame
- added link camera_depth_optical_frame
- added link camera_link, mass 0.001; collision box size=0.015 0.042 0.042; visual box size=0.015 0.042 0.042
Joints:
- added joint camera_color_optical_joint: type fixed, parent camera_link, child camera_color_optical_frame, origin xyz=0 0 0 rpy=-1.5708 0 -1.5708
- added joint camera_depth_optical_joint: type fixed, parent camera_link, child camera_depth_optical_frame, origin xyz=0 0 0 rpy=-1.5708 0 -1.5708
- added joint camera_joint: type fixed, parent gripper_link, child camera_link, origin xyz=0.04 0.0 0.025 rpy=0 1.309 0

File: so-arm/so101_ws/src/so101_moveit_config/config/so101_new_calib.ros2_control.xacro (robot description, xacro)
@@ -1,19 +1,15 @@
 <?xml version="1.0"?>
 <robot xmlns:xacro="http://www.ros.org/wiki/xacro">
-    <xacro:macro name="so101_new_calib_ros2_control" params="name initial_positions_file use_fake_hardware">
+    <xacro:macro name="so101_new_calib_ros2_control" params="name initial_positions_file simulation">
         <xacro:property name="initial_positions" value="${xacro.load_yaml(initial_positions_file)['initial_positions']}"/>
         <ros2_control name="${name}" type="system">
             <hardware>
-                <xacro:if value="${use_fake_hardware}">
-                    <!-- <plugin>mock_components/GenericSystem</plugin> -->
-                    <!-- <plugin>topic_based_ros2_control/TopicBasedSystem</plugin>
-                    <param name="joint_states_topic">/isaac_joint_states</param>
-                    <param name="joint_commands_topic">/isaac_joint_command</param> -->
-                    <plugin>joint_state_topic_hardware_interface/JointStateTopicSystem</plugin>
+                <xacro:if value="${simulation}">
+                    <plugin>topic_based_ros2_control/TopicBasedSystem</plugin>
                     <param name="joint_states_topic">/isaac_joint_states</param>
                     <param name="joint_commands_topic">/isaac_joint_command</param>
                     <param name="sum_wrapped_joint_states">true</param>
                 </xacro:if>
-                <xacro:unless value="${use_fake_hardware}">
+                <xacro:unless value="${simulation}">
                     <plugin>so_arm_100_controller/SOARM100Interface</plugin>
                     <param name="use_serial">true</param>

File: so-arm/so101_ws/src/so101_moveit_config/config/so101_new_calib.urdf.xacro (robot description, xacro)
@@ -2,9 +2,9 @@
 <robot xmlns:xacro="http://www.ros.org/wiki/xacro" name="so101_new_calib">
     <xacro:arg name="initial_positions_file" default="initial_positions.yaml" />
-    <xacro:arg name="use_fake_hardware" default="true" />
+    <xacro:arg name="simulation" default="true" />
     <!-- Import so101_new_calib urdf file -->
     <xacro:include filename="$(find so101_description)/urdf/so101_new_calib.urdf" />
     <!-- Import control_xacro -->
     <xacro:include filename="so101_new_calib.ros2_control.xacro" />
-    <xacro:so101_new_calib_ros2_control name="FakeSystem" initial_positions_file="$(arg initial_positions_file)" use_fake_hardware="$(arg use_fake_hardware)"/>
+    <xacro:so101_new_calib_ros2_control name="SO101System" initial_positions_file="$(arg initial_positions_file)" simulation="$(arg simulation)"/>
 </robot>
